File: QL_nanokeyboard.kicad_pcb (KiCad board)
At the start: 2 copper layers, 94.6 x 54 mm, 20 parts, among them J1 Turned Pins 1x20, J2 Turned Pins 1x20, J9 USB_A, U1 SOCKET 40 PIN, U3 2764, U6 74LS148, U7 74LS14, U8 74LS14

Commit message: add firmware source code
Other:
- board text added: "https://github.com/alvaroalea/QL_Alea_keyboard_interface"
- board text removed: "https://github.com/alvaroalea/QL_nanokeyboard"
