File: QL_nanokeyboard.kicad_sch (KiCad schematic)
At the start: 21 parts, among them J1 Turned Pins 1x20, J2 Turned Pins 1x20, J9 USB_A, U1 SOCKET 40 PIN, U2 GAL16V8, U3 2764, U6 74LS148, U7 74LS14, U8 74LS14

Commit message: add firmware source code
Other:
- title: Unknow Keyboard Interface for Sinclair QL -> USB Keyboard Interface for Sinclair QL
Changed lines of the file:
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@@
 	(paper "A4")
 	(title_block
-		(title "Unknow Keyboard Interface for Sinclair QL")
+		(title "USB Keyboard Interface for Sinclair QL")
 		(date "2024-10-09")
 		(rev "0.1")
